File: hardware/kicad/raccoon-hat.kicad_sch (KiCad schematic)
At the start: 16 parts, among them J1 Conn_02x20_RPi_GPIO, J14 PoE_Header_4pin, J2 HR911105A, J3 USB3_A_Male, T1 750342460, U1 SI3402-B, U2 TPS54302, U3 RTL8153B-VB-CG, U4 AP2112K-3.3, U5 W25Q16JVSSIQ, Y1 25MHz

Commit message: Add functional PCB design, KiCad screenshots, and comprehensive hardware test suite
- Rewrite PCB with proper footprints, pads, traces, and copper zones (KiCad 10 format)
- Add matching schematic with all PoE + USB-to-GbE components
- Add PCB layout screenshot and 3D render to README
- Add 12 hardware tests covering full deployment lifecycle:
  smoke, throughput, power, continuity, bridge transparency,
  cover identity, NAC bypass, OPSEC scan, C2 beacon,
  sniffer/capture, SSH tunnel, and first-boot validation

Co-Authored-By: Claude Opus 4.6 <noreply@anthropic.com>
Parts:
- removed D1: MBRS340, Diode_SMD:D_SMA, symbol Device:D_Schottky
- removed F1: 500mA, Fuse:Fuse_1206_3216Metric, symbol Device:Polyfuse
- removed J1: Conn_02x20_RPi_GPIO, Connector_PinHeader_2.54mm:PinHeader_2x20_P2.54mm_Vertical, symbol Connector_Generic:Conn_02x20_Odd_Even
- removed J14: PoE_Header_4pin, Connector_PinHeader_2.54mm:PinHeader_1x04_P2.54mm_Vertical, symbol Connector_Generic:Conn_01x04
- removed J2: HR911105A, Connector_RJ:RJ45_Amphenol_RJHSE5380, symbol Connector:RJ45_Shielded_MagJack
- removed J3: USB3_A_Male, Connector_USB:USB3_A_Molex_48393, symbol Connector:USB_A
- removed L1: 10uH, Inductor_SMD:L_1210_3225Metric, symbol Device:L
- removed LED1: Green, LED_SMD:LED_0402_1005Metric, symbol Device:LED
- removed LED2: Amber, LED_SMD:LED_0402_1005Metric, symbol Device:LED
- removed T1: 750342460, custom:Transformer_Wuerth_750342460, symbol custom:Transformer_Flyback
- removed U1: SI3402-B, Package_DFN_QFN:QFN-20-1EP_4x4mm_P0.5mm_EP2.5x2.5mm, symbol custom:SI3402-B
- removed U2: TPS54302, Package_TO_SOT_SMD:SOT-23-6, symbol custom:TPS54302
- removed U3: RTL8153B-VB-CG, Package_DFN_QFN:QFN-48-1EP_7x7mm_P0.5mm_EP5.45x5.45mm, symbol custom:RTL8153B-VB-CG
- removed U4: AP2112K-3.3, Package_TO_SOT_SMD:SOT-23-5, symbol Regulator_Linear:AP2112K-3.3
- removed U5: W25Q16JVSSIQ, Package_SO:SOP-8_3.9x4.9mm_P1.27mm, symbol Memory_Flash:W25Q16JV
- removed Y1: 25MHz, Crystal:Crystal_SMD_3215-2Pin_3.2x1.5mm, symbol Device:Crystal
- added C1: 100uF, symbol C
- added C10, C12, C15, C17, C18, C3, C5, C7, C9: 100nF, symbol C
- added C11, C19, C2, C6, C8: 10uF, symbol C
- added C13, C14: 15pF, symbol C
- added C16: 4.7uF, symbol C
- added C4: 22uF, symbol C
- added F1: 500mA, symbol Fuse_PTC
- added J1: GPIO, symbol Conn_02x20_Odd_Even
- added J2: HR911105A, symbol RJ45_Shielded
- added J3: USB-A 3.0, symbol USB_A
- added L1: 10uH, symbol L
- added LED1: Green, symbol LED
- added LED2: Amber, symbol LED
- added R1: 24.9k, symbol R
- added R2: 5.36k, symbol R
- added R3, R4: 330R, symbol R
- added R5: 25.5k, symbol R
- added R6, R7, R8: 10k, symbol R
- added T1: 750342460, symbol Transformer_1P_1S
- added U1: SI3402-B, symbol SI3402-B
- added U2: TPS54302, symbol TPS54302
- added U3: RTL8153B, symbol RTL8153B
- added U4: AP2112K-3.3, symbol AP2112K
- added U5: W25Q16, symbol W25Q16
- added Y1: 25MHz, symbol Crystal
Other:
- company: Raccoon Red Team Hardware -> TrashPandaPaws
- title: Raccoon HAT — PoE Ethernet Tap for Raspberry Pi 4 -> Raccoon HAT v1 — PoE Ethernet Tap
