File: hardware/kicad/raccoon-hat.kicad_pcb (KiCad board)
At the start: 2 copper layers, 65 x 56 mm, 45 parts, among them J1 2x20 GPIO, J2 HR911105A, J3 USB-A 3.0, T1 750342460, U1 SI3402-B, U2 TPS54302, U3 RTL8153B, U4 AP2112K-3.3, U5 W25Q16, Y1 25MHz

Commit message: Audit the v1 HAT hardware and fix the errors found
A structural audit of the KiCad sources and a datasheet review of the chosen
parts. The findings were severe enough that the v1 HAT is now documented as
concept stage rather than buildable. hardware/OPEN_QUESTIONS.md records every
finding with its source.

File state, established by parsing the files (KiCad was not available at the
time, so ERC/DRC could not be run):

  * raccoon-hat.kicad_pcb carried no net table at all and referenced nets by
    name where KiCad requires an integer index, in all 304 places. The file
    would not load. Repaired by tools/fix_pcb_nets.py: a 40-entry net table,
    integer ids on 228 pads and 73 segments, net_name on all 3 zones.
  * raccoon-hat.kicad_sch has effectively no connectivity: 47 symbols but 10
    wires, of which 19 of 20 endpoints land on empty canvas, 7 of 10 wires run
    diagonally, no junctions, no power symbols, and 15 labels none of which
    touch a wire. Netlist export would have been empty.
  * The PCB numbered its resistors R1-R8 where the guide and BOM used R3-R10;
    renumbered to match.

Electrical errors, each verified against the vendor datasheet:

  * R10 feedback divider: the guide assumed a 0.8V reference for the TPS54302
    and derived 19.1K. The real reference is 0.596V (SLVSDF3 6.3.7), so that
    divider yields 3.72V, not 5V, and a Pi 4 would not boot. Now 13.3K, the
    value TI tabulates for 5V. Telling detail: L1, C11+C12 and C1 all already
    matched TI's 5V row, so only the reference had been mis-transcribed.
  * R4 detection resistor was 25.5K, which is the value for the obsolete
    Si3402-A. Skyworks' migration note states it must be 24.3K for the -B.
  * R3 classification resistor was 49.9K. RCLASS is specified in ohms, not
    kilohms; 48.7R selects Class 3, which suits a ~12W PD.
  * R7/R8 LED series resistors were 10k, giving 0.13mA - effectively invisible.
    Now 1K.
  * The Si3402-B symbol matches no Si3402 variant: 0 of 16 pins ag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
Parts:
- renumbered R8 to R10, R1 to R3, R2 to R4, R3 to R5, R4 to R6, R5 to R7, R6 to R8, R7 to R9
